File: CDFR.kicad_pcb (KiCad board)
At the start: 2 copper layers, 56 x 64.9 mm, 20 parts, among them J10_I2C1 Conn_01x04, J1_I2C1 Conn_01x03, J2_I2C1 Conn_01x03, J3_I2C1 Conn_01x03, J4_I2C1 Conn_01x03, J5_I2C1 Conn_01x04, J6 Conn_01x02_Socket, J7 Screw_Terminal_01x02, J8_UART0 Conn_01x05_Socket, J9_I2C1 Conn_01x04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

Commit message: wip
Parts:
- removed D1: D_Zener, Diode_SMD:D_SOD-123
- removed F1: 0154004.DR, FuseHolder:FUSE_0154004.DR
- removed PS2: TEN_15-2411WI, TEN152411:TEN152411WI
- removed Q1: Q_NMOS_GDS, Package_TO_SOT_SMD:TO-252-2
- removed R4: 56k, Resistor_SMD:R_0805_2012Metric_Pad1.20x1.40mm_HandSolder
- added F2: 0154004.DR, footprints:FUSE_0154004.DR, F.Cu at (195.6, 105.4)
- added U2: YAAJ_DCDC_StepDown_LM2596, footprints:YAAJ_DCDC_StepDown_LM2596, F.Cu at (140.0, 44.2)
- J7: footprint TerminalBlockBend:CUI_TBP01R1-508-02BE -> footprints:CUI_TBP01R1-508-02BE
- JP1: value Jumper_3_Open -> Jumper_4_Open; footprint Connector_PinHeader_2.54mm:PinHeader_1x03_P2.54mm_Vertical -> footprints:jumper_4_pole
- R1, R2: footprint Resistor_SMD:R_0805_2012Metric_Pad1.20x1.40mm_HandSolder -> Resistor_SMD:R_0603_1608Metric_Pad0.98x0.95mm_HandSolder
- U1: footprint raspberryPi:EmpreintPourShiel_RaspberryPi3B -> footprints:EmpreintPourShiel_RaspberryPi3B
- moved JP1 64.1 mm to (174.0, 108.6)
- moved U1 0.09 mm to (134.2, 70.9)
Connections:
- J7 pad 1: Net-(J7-Pin_1) -> GND
Routing:
- net +5V: track 151.7 -> 63.7 mm
- net /I2C_SDA: track 181.1 -> 113.7 mm, vias 1 -> 0
- net Net-(J7-Pin_1): track 55.4 -> 0.00 mm, vias 2 -> 0
- net Net-(J7-Pin_2): track 50.1 -> 11.9 mm, vias 2 -> 0
- net Net-(PS2--VIN_(GND)): track 24.0 -> 0.00 mm
- net /I2C_CLK: track 163.0 -> 152.3 mm, vias 2 -> 1
- net Net-(D1-K): track 7.11 -> 0.00 mm
- net GND: track 17.2 -> 23.2 mm

Commit message: wip
Parts:
- added D1: D_Zener, Diode_SMD:D_SOD-123, F.Cu at (144.5, 43.2)
- added Q1: Q_NMOS_GDS, Package_TO_SOT_SMD:TO-252-2, F.Cu at (144.7, 51.1)
- added R4: 56k, Resistor_SMD:R_0603_1608Metric_Pad0.98x0.95mm_HandSolder, F.Cu at (151.8, 37.7)
- R3: footprint Resistor_SMD:R_0805_2012Metric -> Resistor_SMD:R_0603_1608Metric_Pad0.98x0.95mm_HandSolder
- U2: footprint footprints:YAAJ_DCDC_StepDown_LM2596 -> footprints:XL4015-5A
- moved F2 84.4 mm to (147.3, 36.2), turned to -90 degrees
- moved JP1 58.7 mm to (143.5, 58.4)
- moved J7 3.36 mm to (131.1, 38.3)
- moved J8_UART0 1.95 mm to (151.4, 55.8)
- moved J6 1.69 mm to (149.9, 91.4)
- moved U2 1.54 mm to (138.7, 43.3)
- moved R3 1.05 mm to (153.7, 61.5)
- moved R1 0.42 mm to (153.4, 37.8)
- moved R2 0.18 mm to (155.1, 37.7)
Connections:
- J7 pad 1: GND -> Net-(J7-Pin_1)
Routing:
- net +5V: track 63.7 -> 170.7 mm
- net /I2C_SDA: track 113.7 -> 162.3 mm, vias 0 -> 1
- net Net-(J7-Pin_1): track 0.00 -> 21.6 mm
- net Net-(U2-Vin): track 0.00 -> 15.8 mm
- net GND: track 23.2 -> 11.2 mm
- net /I2C_CLK: track 152.3 -> 163.3 mm, vias 1 -> 0
- net Net-(D1-K): track 0.00 -> 10.8 mm
- net Net-(J8_UART0-Pin_5): track 7.81 -> 18.5 mm
- net Net-(J7-Pin_2): track 11.9 -> 16.2 mm
- net MotorControl: track 23.9 -> 26.5 mm
- net Net-(J8_UART0-Pin_3): track 13.2 -> 11.2 mm
- net Net-(J8_UART0-Pin_2): track 12.9 -> 11.3 mm
- net Net-(J6-Pin_1): track 24.3 -> 25.5 mm
