File: CDFR.kicad_sch (KiCad schematic)
At the start: 17 parts, among them J10_I2C1 Conn_01x04, J1_I2C1 Conn_01x03, J2_I2C1 Conn_01x03, J3_I2C1 Conn_01x03, J4_I2C1 Conn_01x03, J5_I2C1 Conn_01x04, J6 Conn_01x02_Socket, J7 Screw_Terminal_01x02, J8_UART0 Conn_01x05_Socket, J9_I2C1 Conn_01x04, U1 RASPBERRY_PI_3_MODEL_B_

Commit message: wip
Parts:
- removed PS2: TEN_15-2411WI, TEN152411:TEN152411WI, symbol SamacSys_Parts:TEN_15-2411WI
- F1: footprint FuseHolder:FUSE_0154004.DR -> footprints:FUSE_0154004.DR
- J7: footprint TerminalBlockBend:CUI_TBP01R1-508-02BE -> footprints:CUI_TBP01R1-508-02BE
- R1, R2: footprint Resistor_SMD:R_0805_2012Metric_Pad1.20x1.40mm_HandSolder -> Resistor_SMD:R_0603_1608Metric_Pad0.98x0.95mm_HandSolder
- U1: footprint raspberryPi:EmpreintPourShiel_RaspberryPi3B -> footprints:EmpreintPourShiel_RaspberryPi3B
Connections:
- no-connect marks 24 -> 23
Changed lines of the file:
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@@
 	)
 	(no_connect
-		(at 63.5 27.94)
-	)
-	(no_connect
 		(at 115.57 86.995)
 	)
@@
 	(label "I2C_CLK"
 		(at 96.52 79.375 0)
-		(fields_autoplaced yes)
 		(effects
 			(font
@@
 	(label "I2C_SDA"
 		(at 95.25 76.835 0)
-		(fields_autoplaced yes)
 		(effects
 			(font
@@
 	)
 	(symbol
-		(lib_id "SamacSys_Parts:TEN_15-2411WI")
-		(at 63.5 27.94 0)
-		(unit 1)
-		(exclude_from_sim no)
-		(in_bom yes)
-		(on_board yes)
-		(dnp no)
-		(fields_autoplaced yes)
-		(property "Reference" "PS2"
-			(at 85.09 20.32 0)
-			(effects
-				(font
-					(size 1.27 1.27)
-				)
-			)
-		)
-		(property "Value" "TEN_15-2411WI"
-			(at 85.09 22.86 0)
-			(effects
-				(font
-					(size 1.27 1.27)
-				)
-			)
-		)
-		(property "Footprint" "TEN152411:TEN152411WI"
-			(at 102.87 122.86 0)
-			(effects
-				(font
-					(size 1.27 1.27)
-				)
-				(justify left top)
-				(hide yes)
-			)
-		)
-		(property "Datasheet" "https://tracopower.com/ten15wi-datasheet/"
-			(at 102.87 222.86 0)
-			(effects
-				(font
-					(size 1.27 1.27)
-				)
-				(justify left top)
-				(hide yes)
-			)
-		)
-		(property "Description" "15 Watt DC/DC converter, industrial, 4:1 input, encapsulated, 2\" x 1\" metal package"
-			(at 63.5 27.94 0)
-			(effects
-				(font
-					(size 1.27 1.27)
-				)
-				(hide yes)
-			)
-		)
-		(property "Height" "10.7"
-			(at 102.87 422.86 0)
-			(effects
-				(font
-					(size 1.27 1.27)
-				)
-				(justify left top)
-				(hide yes)
-			)
-		)
-		(property "Manufacturer_Name" "Traco Power"
-			(at 102.87 522.86 0)
-			(effects
-				(font
-					(size 1.27 1.27)
-				)
-				(justify left top)
-				(hide yes)
-			)
-		)
-		(property "Manufacturer_Part_Number" "TEN 15-2411WI"
-			(at 102.87 622.86 0)
-			(effects
-				(font
-					(size 1.27 1.27)
-				)
-				(justify left top)
-				(hide yes)
-			)
-		)
-		(property "Mouser Part Number" "495-TEN15-2411WI"
-			(at 102.87 722.86 0)
-			(effects
-				(font
-					(size 1.27 1.27)
-				)
-				(justify left top)
-				(hide yes)
-			)
-		)
-		(property "Mouser Price/Stock" "https://www.mouser.co.uk/ProductDetail/TRACO-Power/TEN-15-2411WI?qs=ckJk83FOD0V4P5vtexwoVg%3D%3D"
-			(at 102.87 822.86 0)
-			(effects
-				(font
-					(size 1.27 1.27)
-				)
-				(justify left top)
-				(hide yes)
-			)
-		)
-		(property "Arrow Part Number" ""
-			(at 102.87 922.86 0)
-			(effects
-				(font
-					(size 1.27 1.27)
-				)
-				(justify left top)
-				(hide yes)
-			)
-		)
-		(property "Arrow Price/Stock" ""
-			(at 102.87 1022.86 0)
-			(effects
-				(font
-					(size 1.27 1.27)
-				)
-				(justify left top)
-				(hide yes)
-			)
-		)
-		(pin "6"
-		)
-		(pin "2"
-		)
-		(pin "3"
-		)
-		(pin "1"
-		)
-		(pin "5"
-		)
-		(instances
-			(project ""
-				(path "/4baf3cc7-e737-4c25-a00c-bc79957d9384"
-					(reference "PS2")
-					(unit 1)
-				)
-			)
-		)
-	)
-	(symbol
 		(lib_id "Connector_Generic:Conn_01x03")
 		(at 90.17 76.835 180)
@@
 			)
 		)
-		(property "Footprint" "raspberryPi:EmpreintPourShiel_RaspberryPi3B"
+		(property "Footprint" "footprints:EmpreintPourShiel_RaspberryPi3B"
 			(at 140.97 102.235 0)
 			(effects
@@
 			)
 		)
-		(property "Description" "\nSingle Board Computer, Model B+ 1GB RAM,Raspberry Pi 3 Series | Raspberry Pi RASPBERRY PI 3 MODEL B+\n"
+		(property "Description" "Single Board Computer, Model B+ 1GB RAM,Raspberry Pi 3 Series | Raspberry Pi RASPBERRY PI 3 MODEL B+"
 			(at 140.97 102.235 0)
 			(effects
@@
 			)
 		)
-		(property "Footprint" "TerminalBlockBend:CUI_TBP01R1-508-02BE"
+		(property "Footprint" "footprints:CUI_TBP01R1-508-02BE"
 			(at 38.1 27.94 0)
 			(effects
@@
 			)
 		)
-		(property "Footprint" "FuseHolder:FUSE_0154004.DR"
+		(property "Footprint" "footprints:FUSE_0154004.DR"
 			(at 55.88 48.26 0)
 			(effects
@@
 			)
 		)
-		(property "Footprint" "Resistor_SMD:R_0805_2012Metric_Pad1.20x1.40mm_HandSolder"
+		(property "Footprint" "Resistor_SMD:R_0603_1608Metric_Pad0.98x0.95mm_HandSolder"
 			(at 104.902 80.645 90)
 			(effects
@@
 			)
 		)
-		(property "Footprint" "Resistor_SMD:R_0805_2012Metric_Pad1.20x1.40mm_HandSolder"
+		(property "Footprint" "Resistor_SMD:R_0603_1608Metric_Pad0.98x0.95mm_HandSolder"
 			(at 97.282 83.185 90)
 			(effects

Commit message: wip
Parts:
- removed F1: 0154004.DR, footprints:FUSE_0154004.DR, symbol 0154004.DR:0154004.DR
- removed JP1: Jumper_3_Open, Connector_PinHeader_2.54mm:PinHeader_1x03_P2.54mm_Vertical, symbol Jumper:Jumper_3_Open
- removed U1: RASPBERRY_PI_3_MODEL_B_, footprints:EmpreintPourShiel_RaspberryPi3B, symbol RASPBERRY_PI_3_MODEL_B_:RASPBERRY_PI_3_MODEL_B_
- added F2: 0154004.DR, footprints:FUSE_0154004.DR, symbol symbols:0154004.DR
- added JP1: Jumper_4_Open, footprints:jumper_4_pole, symbol symbols:Jumper_4_Open
- added U1: RASPBERRY_PI_3_MODEL_B_, footprints:EmpreintPourShiel_RaspberryPi3B, symbol symbols:RASPBERRY_PI_3_MODEL_B_
- added U2: YAAJ_DCDC_StepDown_LM2596, footprints:YAAJ_DCDC_StepDown_LM2596, symbol symbols:YAAJ_DCDC_StepDown_LM2596
Connections:
- net +3.3V: now also U1.1 (3V3)
- net +5V: now also JP1.1 (A), U1.2 (5V), U1.4 (5V), U2.4 (Vout)
- net GND: now also J7.1 (Pin_1), JP1.5 (A), U1.14 (GND), U1.20 (GND), U1.25 (GND), U1.30 (GND), U1.34 (GND), U1.39 (GND), U1.6 (GND), U1.9 (GND), U1.S1 (SHIELD), U1.S2 (SHIELD), U1.S3 (SHIELD), U1.S4 (SHIELD), U2.2 (GND), U2.3 (GND)
- net I2C_CLK: now also U1.5 (GPIO3/SCL1)
- net I2C_SDA: now also U1.3 (GPIO2/SDA1)
- net MotorControl: now also JP1.3 (B), U1.12 (GPIO18/GPIO_GEN1)
- net at J6.1 (Pin_1): now also U1.29 (GPIO5)
- net at J8_UART0.2 (Pin_2): now also U1.10 (GPIO15/RXD0)
- net at J8_UART0.3 (Pin_3): now also U1.8 (GPIO14/TXD0)
- net at J8_UART0.5 (Pin_5): now also JP1.2 (C)
- net at J7.2 (Pin_2): now also F2.1
- new net: F2.2, U2.1 (Vin)
- no-connect marks 23 -> 24
Other:
- moved on the sheet: J10_I2C1, J1_I2C1, J2_I2C1, J3_I2C1, J4_I2C1, J5_I2C1, J7, J8_UART0, J9_I2C1, R1, R2, R3

Commit message: wip
Parts:
- added D1: D_Zener, Diode_SMD:D_SOD-123, symbol Device:D_Zener
- added Q1: Q_NMOS_GDS, Package_TO_SOT_SMD:TO-252-2, symbol Device:Q_NMOS_GDS
- added R4: 56k, Resistor_SMD:R_0603_1608Metric_Pad0.98x0.95mm_HandSolder, symbol Device:R
- R3: footprint Resistor_SMD:R_0805_2012Metric -> Resistor_SMD:R_0603_1608Metric_Pad0.98x0.95mm_HandSolder
Connections:
- net GND: now also D1.2 (A), Q1.3 (S); no longer J7.1 (Pin_1)
- net at F2.2, U2.1 (Vin): now also R4.1
- new net: J7.1 (Pin_1), Q1.2 (D)
- new net: D1.1 (K), Q1.1 (G), R4.2
Other:
- moved on the sheet: F2, J7
